File: CAD/KiCAD/stm32f401cc/stm32f401cc.kicad_sch (KiCad schematic)
At the start: 11 parts, among them U1 STM32F401CCUx, Y1 25MHz, Y2 32.768kHz

Commit message: acquire
Parts:
- removed C1, C2: C_Small, Capacitor_SMD:C_0201_0603Metric, symbol Device:C_Small
- removed Y2: 32.768kHz, Crystal:Crystal_SMD_2012-2Pin_2.0x1.2mm_HandSoldering, symbol Device:Crystal_Small
